File: hardware/safekiln.kicad_sch (KiCad schematic)
At the start: 117 parts, among them J1 5V DC IN, J10 CT 30A/1V (opt), J11 UART / EXPANSION, J2 USB-C, J3 TC1 KILN (K), J4 TC2 CASE (K), J5 OLED 128x64 I2C, J6 SSR1 CTRL, J8 CONTACTOR COIL 5V, J9 LID SWITCH, Q1 AO3400A, Q3 AO3400A, Q4 AO3400A, Q5 AO3400A, Q6 AO3400A, SW1 RESET, SW2 BOOT, SW3 ENCODER, U1 ESP32-S3-WROOM-1, U2 AMS1117-3.3, U3 MAX31856, U4 MAX31856

Commit message: chore: the kicad project is safekiln, and the fixture follows it
The board, schematic and project file are renamed from kilncontrol to
safekiln, matching what the firmware, the image and the documentation have
called this product since the repository was reorganised.

Three references had to move with it, and they are the ones that would have
failed silently rather than loudly:

  fixture/pinside-baseline.json names the board it is a baseline OF, so a
  rename without it means `pinside check` has nothing to compare against.

  fixture/kilncontrol-fixture.json carries an absolute path to the board. It
  keeps its own filename: that is the fixture's name, not the project's, and
  renaming an input this project owns is a separate decision from renaming the
  board.

  fixture/README.md documents the command a person types.

Not touched: fixture/firmware/ and fixture/board/, which pinside generates
verbatim and will rewrite from the new name on the next run, and which CI
already excludes from the SPDX check for the same reason.
Parts:
- removed J4: TC2 CASE (K), TerminalBlock:TerminalBlock_MaiXu_MX126-5.0-02P_1x02_P5.00mm, symbol Connector:Screw_Terminal_01x02
- removed Q6: AO3400A, Package_TO_SOT_SMD:SOT-23, symbol Transistor_FET:Q_NMOS_GSD
- removed R28: 10k, Resistor_SMD:R_0402_1005Metric, symbol Device:R
- removed TP11: TC1_DRDY, TestPoint:TestPoint_Pad_1.5x1.5mm, symbol Connector:TestPoint
- removed TP22: COIL_DRV, TestPoint:TestPoint_Pad_1.5x1.5mm, symbol Connector:TestPoint
- removed TP4: GND, TestPoint:TestPoint_Pad_1.5x1.5mm, symbol Connector:TestPoint
- removed TP5: VBUS, TestPoint:TestPoint_Pad_1.5x1.5mm, symbol Connector:TestPoint
- added C26: 100nF, Capacitor_SMD:C_0402_1005Metric, symbol Device:C
- added C27: 10uF, Capacitor_SMD:C_0805_2012Metric, symbol Device:C
- added D4: BAT54C, Package_TO_SOT_SMD:SOT-23, symbol Diode:BAT54C
- added J4: Conn_ARM_SWD_TagConnect_TC2030, Connector:Tag-Connect_TC2030-IDC-NL_2x03_P1.27mm_Vertical, symbol Connector:Conn_ARM_SWD_TagConnect_TC2030
- added J7: TC2 KILN (K), TerminalBlock:TerminalBlock_MaiXu_MX126-5.0-02P_1x02_P5.00mm, symbol Connector:Screw_Terminal_01x02
- added R16, R17: 100R, Resistor_SMD:R_0402_1005Metric, symbol Device:R
- added R32: 10k, Resistor_SMD:R_0402_1005Metric, symbol Device:R
- added R33: 18k, Resistor_SMD:R_0402_1005Metric, symbol Device:R
- added TP34: COIL_PERMIT, TestPoint:TestPoint_Pad_1.5x1.5mm, symbol Connector:TestPoint
- added TP35: SUPERVISOR_TX, TestPoint:TestPoint_Pad_1.5x1.5mm, symbol Connector:TestPoint
- added TP36: SUPERVISOR_RESET, TestPoint:TestPoint_Pad_1.5x1.5mm, symbol Connector:TestPoint
- added TP37: COIL_FEEDBACK, TestPoint:TestPoint_Pad_1.5x1.5mm, symbol Connector:TestPoint
- added TP38: TC2_N, TestPoint:TestPoint_Pad_1.5x1.5mm, symbol Connector:TestPoint
- added U5: STM32G031K8Tx, Package_QFP:LQFP-32_7x7mm_P0.8mm, symbol MCU_ST_STM32G0:STM32G031K8Tx
- C14: value 10nF -> 100nF; LCSC C15195 -> C1525
- C15: value 100pF -> 100nF; LCSC C26409 -> C1525
- C16: value 100pF -> 10nF; LCSC C26409 -> C15195
- C17, C18: value 100nF -> 100pF; LCSC C1525 -> C26409
- C19: value 10uF -> 100nF; footprint Capacitor_SMD:C_0805_2012Metric -> Capacitor_SMD:C_0402_1005Metric; LCSC C15850 -> C1525
- D3, TP17: value SSR1 -> SSR
- J10: value CT 30A/1V (opt) -> CT 30A/1V
- J6: value SSR1 CTRL -> SSR CTRL
- R6: value 100R -> 220R
- R7: value 100R -> 10k
- TP10: value TC2_CS -> TC2_SCK
- TP12: value TC2_DRDY -> TC2_MOSI
- TP14: value TC2_FAULT -> TC2_MISO
- TP18: value SSR2 -> TC2_CS
- TP30: value TC2_N -> TC2_FAULT
- TP32: value MCU_EN -> ESP32_EN
- TP33: value MCU_IO0 -> ESP32_IO0
- TP6: value SPI_SCK -> TC1_SCK
- TP7: value SPI_MOSI -> TC1_MOSI
- TP8: value SPI_MISO -> TC1_MISO
Connections:
- net +3V3 is gone; now on net +3.3V: TP2.1
- net COIL_RTN2 is gone; now on net COIL_RTN1: Q5.3 (D)
- net +3.3V: now also C14.1, R7.2, C26.1, C27.1, J4.1 (VCC), U5.4 (VDD); no longer C17.1, C18.1
- net COIL_DRV: now also R32.1
- net GND: now also C14.2, C26.2, C27.2, J4.5 (GND), R33.2, U5.5 (VSS); no longer C16.2
- net TC1_CS: now also U5.11 (PA4); no longer U1.18 (IO10)
- net TC1_FAULT: now also U5.10 (PA3)
- net TC1_N: now also U3.2 (BIAS)
- net TC1_TN: no longer U3.2 (BIAS)
- net TC2_CS: now also TP18.1, U5.29 (PB5); no longer TP10.1, U1.17 (IO9)
- net TC2_FAULT: now also TP30.1, U5.28 (PB4); no longer Q5.1 (G), R29.2, TP14.1
- net TC2_N: now also U4.2 (BIAS), J7.1 (Pin_1), R17.1, TP38.1; no longer R7.1, TP30.1
- net TC2_P: now also J7.2 (Pin_2), R16.1; no longer R6.1
- net TC2_TN: now also C16.2, C18.1, R17.2; no longer C14.2, C16.1, R7.2, U4.2 (BIAS)
- net TC2_TP: now also C16.1, C17.1, R16.2; no longer C14.1, C15.1, R6.2
- net SUPERVISOR_TX: now reaches U1.24 (IO47)
- net SUPERVISOR_TX: now also R6.2, R7.1, J4.6 (SWO), TP35.1
- net MCU_EN renamed ESP32_EN
- net ESP32_EN: now also D4.2; no longer SW1.2
- net MCU_IO0 renamed ESP32_IO0
- net SPI_MISO renamed TC1_MISO
- net TC1_MISO: now also U5.13 (PA6); no longer U1.21 (IO13), U4.11 (SDO)
- net SPI_MOSI renamed TC1_MOSI
- net TC1_MOSI: now also U5.14 (PA7); no longer U1.19 (IO11), U4.12 (SDI)
- net SPI_SCK renamed TC1_SCK
- net TC1_SCK: now also U5.12 (PA5); no longer U1.20 (IO12), U4.10 (SCK)
- net SSR1 renamed SSR
- net SSR1_DRV renamed SSR_DRV
- net SSR2: no longer names the net of U1.5 (IO5)
- net SSR2: no longer TP18.1
- net TC1_DRDY: no longer names the net of U1.22 (IO14)
- net TC1_DRDY: no longer U3.7 (~{DRDY})
- removed net TC2_DRDY: TP12.1, U1.23 (IO21), U4.7 (~{DRDY})
- net USB_DM renamed USB_DN
- new net: R6.1, U5.9 (PA2)
- new net: D4.3, SW1.2
- new net COIL_FEEDBACK: R32.2, R33.1, TP37.1, U5.8 (PA1)
- new net COIL_PERMIT: Q5.1 (G), R29.2, TP34.1, U5.18 (PA8)
- new net SUPERVISOR_RESET: C15.1, D4.1, J4.3 (~{RESET}), TP36.1, U5.7 (PA0)
- new net SW_CLK: J4.4 (SWCLK), U5.25 (PA14)
- new net SW_DIO: J4.2 (SWDIO), U5.24 (PA13)
- new net TC2_MISO: TP14.1, U4.11 (SDO), U5.30 (PB6)
- new net TC2_MOSI: TP12.1, U4.12 (SDI), U5.31 (PB7)
- new net TC2_SCK: TP10.1, U4.10 (SCK), U5.32 (PB8)
- no-connect marks 14 -> 32
Other:
- note added: "SUPERVISOR"
- note added: "The CT must be a voltage-output type with an integral burden resistor; a current-output CT whose burden can be disconnected develops dangerous voltages on an open secondary."
- note removed: "KNOWN ACCEPTED ERC VIOLATION: U3.SDO and U4.SDO both sit on SPI_MISO. The KiCad symbol types these pins "output", but the MAX31856 tri-states SDO whenever its CS is de-asserted, so the shared bus is correct. Separate CS lines (TC1_CS / TC2_CS) guarantee only one device drives at a time. Exclude in ERC."
- title: Main -> Safe Kiln
- moved on the sheet: BZ1, C10, C11, C12, C13, C20, C21, C22, C25, C8, C9, D3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

Commit message: feat: a part number on every bom line, and the buttons go surface mount
Includes the J3/J7 split made in the editor: the two thermocouples are two
2-position blocks again rather than one 4-way, which is what the catalogue
actually stocks. LCSC lists KF301-5.0 in 2P and 3P and no 4P, so the
consolidated connector was a part nobody could order.

All 90 BOM lines now carry an LCSC number, 34 distinct, with the 34 test
points and J4 excluded as the bare pads they are rather than appearing as
lines a BOM cannot fulfil. Three defects came out of doing it:

  R6 and R7 both carried C25076, which is a 100R resistor, while R6 is 220R
  and R7 is 10k. R7 is the pull-up in the supervisor's TX network, so 100R
  would have drawn 33 mA and left R6 no longer limiting anything. One part
  number had propagated onto three different resistance values by field copy.
  Now C25091 and C25744.

  J7 kept J3's value when it was copied, so both thermocouple blocks read
  TC1, on the BOM and on the silkscreen, for a board whose two couples are
  the thing the supervisor cross-checks.

  The 34 test points were (in_bom yes).

Nothing caught any of that because there is no hardware gate in CI at all:
no ERC, no DRC, no BOM check. ERC is clean today at --severity-all with no
exclusions, and tools/fetch3d.py --check verifies the models, so a job
running both plus "every BOM line has an LCSC" and "no part number against
two values" would hold the line at no cost. Tracked as A33.

SW1, SW2 and BZ1 are surface mount. The switches go to the XKB TS-1187A
(C318884), whose footprint KiCad already ships, and neither switch net was
routed yet, so the swap cost no rework. The low-profile 1.5 mm variant is
deliberate: these are service controls, and while RESET also clears the
supervisor's trip latch through D4 (A27), making it easier to press by
accident would be a step backwards.

BZ1 goes to the FST-9650B-5V (C391033), which keeps SYS-HW-09 as written:
active with built-in drive, magnetic, 5 V, and th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
Parts:
- BZ1: value TMB12A05 5V -> FST-9650B 5V; footprint Buzzer_Beeper:Buzzer_12x9.5RM7.6 -> safekiln:Buzzer_FUET_FST-9650B-5V_9.6x9.6mm; LCSC C96093 -> C391033
- D4: LCSC (none) -> C236933
- J3: value TC1 KILN (K) -> TC1
- J7: value TC2 KILN (K) -> TC2
- Q5: LCSC (none) -> C20917
- R29, R30, R32: LCSC (none) -> C25744
- R31, R33: LCSC (none) -> C25762
- R6: LCSC C25076 -> C25091
- R7: LCSC C25076 -> C25744
- SW1, SW2: footprint Button_Switch_THT:SW_PUSH_6mm_H5mm -> Button_Switch_SMD:SW_Push_1P1T_XKB_TS-1187A; LCSC C111609 -> C318884
- TP1, TP10, TP12, TP13, TP14, TP15, TP16, TP17, TP18, TP19, TP2, TP20, TP21, TP23, TP24, TP25, TP26, TP27, TP28, TP29, TP3, TP30, TP31, TP32, TP33, TP34, TP35, TP36, TP37, TP38, TP6, TP7, TP8, TP9: now left out of the parts list
- U5: LCSC (none) -> C432203
Connections:
- net +3.3V: no longer R29.1
- net COIL_PERMIT: now also R29.1; no longer R29.2
- net GND: now also R29.2
- net TC1_N: now also J3.2 (Pin_2); no longer J3.1 (Pin_1)
- net TC1_P: now also J3.1 (Pin_1); no longer J3.2 (Pin_2)
- net TC2_N: now also J7.2 (Pin_2); no longer J7.1 (Pin_1)
- net TC2_P: now also J7.1 (Pin_1); no longer J7.2 (Pin_2)
Other:
- note added: "ALARM"
- note removed: "AUX"
- moved on the sheet: BZ1, D8, Q4, R22, R23

Commit message: feat: a 12 V board with a buck, and the lid input that could not see the lid
The board takes 12 V in and drives a 12 V contactor coil. The +5V rail is
now +12V, and the AMS1117 is gone: at 12 V in it would have dropped 8.7 V
linearly, 2.6 W at 300 mA in a SOT-223. U2 is a TPS54202 (4.5 to 28 V, 2 A,
C191884) with L1 10 uH, 2 x 22 uF out and R34/R35 setting 3.29 V. HWR-14 and
HWR-15 are rewritten for it, and SYS-HW-14 says 12 V.

USB is data only. VBUS was diode-OR'd onto the supply, which on 12 V would
have made a half-powered board: logic running from a USB host, the SSR input
able to switch, the coil unable to pull in and the buzzer silent. D2 is gone
and VBUS goes nowhere. D1 stays, because J1 is a screw terminal and reverse
polarity is the likeliest wiring mistake there is.

Parts that could not live on 12 V: F1 was a 6 V PTC (now 1.1 A / 16 V), C1 a
16 V electrolytic (now 25 V), R15 and R21 1k in 0402 (now 2.2k in 0603), and
BZ1 a 5 V buzzer. There is no 12 V version of the 9.6 mm SMD part, so BZ1 is
a TMB12A12, through-hole and 9.5 mm tall. That undoes the SMD buzzer of
0b7f360, and the enclosure's h_buzzer still says 5.5. SYS-HW-09 now says
12 V.

A review of the result found three defects, two of them older than today:

  The supervisor's reset was on PA0. SUPERVISOR_RESET (J4 RESET, C15, D4)
  went to U5 pin 7 and pin 6, PF2/NRST, was open, so the debugger could not
  reset the supervisor, SW1 reset the ESP32-S3 alone, and the clear button
  pins.h puts on PA0 did not exist. Reset is on pin 6 now, and SW4 CLEAR
  with TP39 is on PA0 (SUP_CLEAR), wired to nothing else, as HWR-19 asks.

  The COIL LED bypassed the lid contact. R21 was fed from the supply, so with
  the lid open and both series elements off, current ran R21 -> D7 ->
  COIL_DRV -> D6 -> LID_SWITCH and put about 2 V on LID_SENSE, between the
  ESP32-S3's thresholds. An open lid could read shut, and COIL_FEEDBACK read
  high whatever the lid did. The interlock held, since an LED's milliamps
  can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
Parts:
- removed D2: SS34, Diode_SMD:D_SMA, symbol Device:D_Schottky
- removed U2: AMS1117-3.3, Package_TO_SOT_SMD:SOT-223-3_TabPin2, symbol Regulator_Linear:AMS1117-3.3
- added C28: 100nF, Capacitor_SMD:C_0402_1005Metric, symbol Device:C
- added C29: 22uF, Capacitor_SMD:C_0805_2012Metric, symbol Device:C
- added C30: 100nF 50V, Capacitor_SMD:C_0603_1608Metric, symbol Device:C
- added C31: 10uF, Capacitor_SMD:C_0805_2012Metric, symbol Device:C
- added C32: 4.7uF, Capacitor_SMD:C_0603_1608Metric, symbol Device:C
- added D10: BAT54S, Package_TO_SOT_SMD:SOT-23, symbol Diode:BAT54S
- added D11: SMBJ15CA, Diode_SMD:D_SMB, symbol Device:D_TVS
- added F2: PTC 0.5A 15V, Fuse:Fuse_1206_3216Metric, symbol Device:Fuse
- added H1, H2, H3, H4: Mount, MountingHole:MountingHole_3.2mm_M3_ISO7380_Pad, symbol Mechanical:MountingHole_Pad
- added L1: 10uH, Inductor_SMD:L_Sunlord_SWPA5040S, symbol Device:L
- added R34: 100k, Resistor_SMD:R_0402_1005Metric, symbol Device:R
- added R35: 22.1k, Resistor_SMD:R_0402_1005Metric, symbol Device:R
- added SW4: CLEAR, Button_Switch_SMD:SW_Push_1P1T_XKB_TS-1187A, symbol Switch:SW_Push
- added TP39: SUP_CLEAR, TestPoint:TestPoint_Pad_1.5x1.5mm, symbol Connector:TestPoint
- added U2: TPS54202DDCR, Package_TO_SOT_SMD:SOT-23-6, symbol Regulator_Switching:TPS54202DDC
- added U6: USBLC6-2SC6, Package_TO_SOT_SMD:SOT-23-6, symbol Power_Protection:USBLC6-2SC6
- BZ1: value FST-9650B 5V -> TMB12A12; footprint safekiln:Buzzer_FUET_FST-9650B-5V_9.6x9.6mm -> Buzzer_Beeper:Buzzer_12x9.5RM7.6; LCSC C391033 -> C96079
- C1: value 100uF 16V -> 100uF 25V; LCSC C231174 -> C176675
- C3: value 10uF -> 22uF; LCSC C15850 -> C45783
- D6: value 1N4148W -> SS14; footprint Diode_SMD:D_SOD-123 -> Diode_SMD:D_SMA; LCSC C2099 -> C2480
- F1: value PTC 1.5A -> PTC 1.1A 16V; LCSC C20802 -> C7542961
- J1: value 5V DC IN -> 12V DC IN
- J5: footprint Connector_PinHeader_2.54mm:PinHeader_1x04_P2.54mm_Vertical -> Connector_PinSocket_2.54mm:PinSocket_1x04_P2.54mm_Vertical; LCSC C2691448 -> (none)
- J8: value CONTACTOR COIL 5V -> CONTACTOR COIL 12V
- R15, R21: value 1k -> 2.2k; footprint Resistor_SMD:R_0402_1005Metric -> Resistor_SMD:R_0603_1608Metric; LCSC C11702 -> C4190
- R30: value 10k -> 22k; LCSC C25744 -> C25768
- R31, R33: value 18k -> 10k; LCSC C25762 -> C25744
- R32: value 10k -> 33k; LCSC C25744 -> C25779
- TP1: value +5V -> +12V
Connections:
- net +3.3V: now also C29.1, C32.1, D10.2 (K), L1.2, R34.1
- net GND: now also C29.2, C30.2, C31.2, C32.2, D10.1 (A), D11.1 (A1), H1.1, H2.1, H3.1, H4.1, R35.2, SW4.1, U2.1 (GND), U6.2 (GND)
- net LID_SENSE: now also D10.3 (COM)
- net LID_SWITCH: now also R21.1
- net SUPERVISOR_RESET: now also U5.6 (PF2); no longer U5.7 (PA0)
- net USB_DN: now also U6.3 (I/O2), U6.4 (I/O2)
- net USB_DP: now also U6.1 (I/O1), U6.6 (I/O1)
- net VBIAS: now also C31.1
- net V_FUSED: now also D11.2 (A2)
- net +5V renamed +12V
- net +12V: now also C30.1, F2.1, U2.3 (VIN); no longer J9.1 (Pin_1), R21.1
- net VBUS: no longer names the net of J2.A4 (VBUS), J2.A9 (VBUS), J2.B4 (VBUS), J2.B9 (VBUS)
- new net: R34.2, R35.1, U2.4 (FB)
- new net: C28.1, L1.1, U2.2 (SW)
- new net: C28.2, U2.6 (BOOT)
- new net: F2.2, J9.1 (Pin_1)
- new net SUP_CLEAR: SW4.2, TP39.1, U5.7 (PA0)
- no-connect marks 32 -> 34
Other:
- moved on the sheet: C1, C2, C3, C4, J1

Commit message: fix: the fault lines get pull-ups, and DRDY is written down as unused
HWR-06 asked for a pull-up on every MAX31856 ~DRDY and ~FAULT, and the board
had none. ~FAULT relied on the supervisor's internal pull-ups on PA3 and PB4,
which exist only once its firmware has configured the pins, so through reset,
through boot and for a supervisor that never gets that far the lines floated,
and an open-drain fault output reads as asserted when it floats. R36 and R37,
10k (C25744), now hold TC1_FAULT and TC2_FAULT to +3V3 beside U3 and U4.

~DRDY gets no resistor because nothing reads it. The supervisor runs both
parts in continuous conversion and takes temperature and fault status in one
burst, and at start-up it waits for the first conversion by reading the
registers rather than the pin. Both ~DRDY pins already carried a no-connect
flag. HWR-06 now says so instead of asking for a pull-up that would serve
nothing, and HWR-05 and SYS-HW-02, which listed ~DRDY among the lines the two
front ends must not share, list ~FAULT and point at HWR-06.

Verified: ERC 0 violations, 108 nets and 384 nodes with each fault net running
pull-up, test point, MAX31856, STM32; StrictDoc 0.30.1 exports clean.
Parts:
- added R36, R37: 10k, Resistor_SMD:R_0402_1005Metric, symbol Device:R
Connections:
- net +3.3V: now also R36.1, R37.1
- net TC1_FAULT: now also R36.2
- net TC2_FAULT: now also R37.2

Commit message: feat: the board catches up with the 12 V schematic
Update PCB from Schematic, run in the editor: the buck (U2, L1, C28 to C30),
U6, D10, D11, F2, SW4, R36/R37, C31/C32, TP39 and the new footprints for U2,
BZ1, D6, R15 and R21 are on the board. The schematic gains TP4, a second GND
test point, and is otherwise electrically unchanged.

DRC with --schematic-parity: 0 unconnected pads and 0 footprint errors, down
from 61 unconnected pads, so the board and the schematic agree. 209
violations remain, against 232 before, and 199 of them are silkscreen
overlaps. What is left that is not cosmetic:

  J2's stacked VBUS pads (A4/B9 and A9/B4) report as shorts and mask
  bridges, two of each. VBUS is unconnected in the schematic, so each pad
  gets its own "unconnected-" net and the pads that share copper look like
  two nets touching. Naming the net fixes it, and lets U6 pin 5 take VBUS
  as the USBLC6 expects.

  One dangling 0.625 mm +12V stub at 144.1, 55.1, and one starved thermal.

  U1's footprint differs from the RF_Module library copy.

Adds safekiln.kicad_dru, the project's custom design rules, and
safekiln.xml, an IPC-2581 export of the board.
Parts:
- added TP4: GND, TestPoint:TestPoint_Pad_1.5x1.5mm, symbol Connector:TestPoint
Connections:
- net GND: now also TP4.1
Other:
- moved on the sheet: TP3
